File: CoilDriver_v0.1/CoilDriver_v0.1.kicad_pcb (KiCad board)
At the start: 4 copper layers, 163 x 100 mm, 217 parts, among them CN1 C3697-WJ2EDGRC-5.08-02P-14-00A, CN2 C71370-WJ2EDGK-5.08-02P-14-00A, CN3 C3697-WJ2EDGRC-5.08-02P-14-00A, CN4 C71370-WJ2EDGK-5.08-02P-14-00A, CN5 C3697-WJ2EDGRC-5.08-02P-14-00A, CN6 C71370-WJ2EDGK-5.08-02P-14-00A, CN7 C3697-WJ2EDGRC-5.08-02P-14-00A, CN8 C71370-WJ2EDGK-5.08-02P-14-00A, J1 C5173361-DIN41612-CONN-TH_96P, J2 Conn_01x02, J3 C306220-826925-6, SW1 C458084-DS-08RP, T1 C7220836-BSC010N04LS6ATMA1, T10 C7220836-BSC010N04LS6ATMA1, T11 C7220836-BSC010N04LS6ATMA1, T12 C7220836-BSC010N04LS6ATMA1, T2 C7220836-BSC010N04LS6ATMA1, T3 C7220836-BSC010N04LS6ATMA1, T4 C7220836-BSC010N04LS6ATMA1, T5 C7220836-BSC010N04LS6ATMA1, T6 C7220836-BSC010N04LS6ATMA1, T7 C7220836-BSC010N04LS6ATMA1, T8 C7220836-BSC010N04LS6ATMA1, T9 C7220836-BSC010N04LS6ATMA1, U1 C2687965-OPA548FKTWT, U10 C2071868-AP63200WU-7, U11 C2071868-AP63200WU-7, U12 C50793 - NC7WZ14P6X, U13 C2653336-74FCT521CTSOG8, U14 C114502 - M24C02-FDW, U15 C22461594 - PCF8574AP, U16 C22469958 - 74LVC1GU04, U17 C113280 - SN74LVC573APWR, U18 C7835-SN74LVC1G14DBVR, U19 C637542-MIC4428YM, U2 C506609-SISS27DN-T1-GE3, U20 C259972-LM1084S-3.3_TR, U21 C1855802-INA293B2IDBVR, U22 C2687965-OPA548FKTWT, U23 C550069-BZB784-C15,115, U24 C637542-MIC4428YM, U25 C1855802-INA293B2IDBVR, U26 C2687965-OPA548FKTWT, U27 C550069-BZB784-C15,115, U28 C637542-MIC4428YM, U3 C1855802-INA293B2IDBVR, U4 C550069-BZB784-C15,115, U5 C207245-SD15C-01FTG, U6 C1554484-DAC8555IPW, U7 C157411-LD29150DT50R, U8 C659573-ADR443BRZ-REEL7, U9 C907854-SD12C

Commit message: Commit Fixes
Parts:
- removed G1: IAMSnanofiber, IAMS:IAMSnanofiber
- removed G2: IAMS, IAMS:IAMS
- removed G3: IAMSYb, IAMS:IAMSYb
