File: CoilDriver_v0.1/CoilDriver_v0.1.kicad_sch (KiCad schematic)
At the start: 33 parts, among them CN1 C3697-WJ2EDGRC-5.08-02P-14-00A, CN2 C71370-WJ2EDGK-5.08-02P-14-00A, CN3 C3697-WJ2EDGRC-5.08-02P-14-00A, CN4 C71370-WJ2EDGK-5.08-02P-14-00A, CN5 C3697-WJ2EDGRC-5.08-02P-14-00A, CN6 C71370-WJ2EDGK-5.08-02P-14-00A, CN7 C3697-WJ2EDGRC-5.08-02P-14-00A, CN8 C71370-WJ2EDGK-5.08-02P-14-00A, J1 C5173361-DIN41612-CONN-TH_96P, J2 Conn_01x02, SW1 C458084-DS-08RP, U12 C50793 - NC7WZ14P6X, U13 C2653336-74FCT521CTSOG8, U14 C114502 - M24C02-FDW, U15 C22461594 - PCF8574AP, U16 C22469958 - 74LVC1GU04, U17 C113280 - SN74LVC573APWR

Commit message: Commit Fixes
Parts:
- removed G1: IAMSnanofiber, IAMS:IAMSnanofiber, symbol IAMS:IAMSnanofiber
- removed G2: IAMS, IAMS:IAMS, symbol IAMS:IAMS
- removed G3: IAMSYb, IAMS:IAMSYb, symbol IAMS:IAMSYb
